File: pcb/NourK/NourK.kicad_pcb (KiCad board)
At the start: 4 copper layers, 304 x 240 mm, 184 parts, among them IC1 IS31FL3733B-QFLS4-TR, J1 SJ-435107RS, J2 Conn_ARM_JTAG_SWD_10, J3 USB_C_Receptacle_USB2.0, J4 USB_C_Receptacle_USB2.0, J5 SJ-435107RS, SW1 SW_SPST_G, SW10 LAYER, SW11 I, SW12 K, SW13 ,, SW14 LAYER, SW15 O, SW16 L, SW17 ., SW18 LAYER, SW19 P, SW2 SW_SPST_G, SW20 ;, SW21 /, SW22 RCTRL, SW23 [, SW24 ', SW25 RSHIFT, SW26 ], SW27 ENTER, SW3 Y, SW30 ESCAPE, SW31 OSKEY, SW32 TAB, SW33 GRAVE, SW34 LEFT_SHIFT, SW35 Q, SW36 A, SW37 Z, SW38 LEFT_CTRL, SW39 W, SW4 H, SW40 S, SW41 X, SW42 LAYER1, SW43 E, SW44 D, SW45 C, SW46 LAYER2, SW47 R, SW48 F, SW49 V, SW5 N, SW50 LEFT_ALT, SW51 T, SW52 G, SW53 B, SW54 SPACE, SW6 SPACE, SW7 U, SW8 J, SW9 M, U1 STM32L082CZYx, U2 AP2112K-3.3, U3 NourK_Core, U4 NourK_Core, U5 NourK_Core, Y1 32.768KHz, Y2 8MHz

Commit message: Draft wire the core
Parts:
- added C21: 100nF, Capacitor_SMD:C_0805_2012Metric, F.Cu at (15.8, 30.0)
- added R13: 5K1, Resistor_SMD:R_0805_2012Metric, F.Cu at (26.0, 52.8)
- added R14: 5K1, Resistor_SMD:R_0805_2012Metric, F.Cu at (30.4, 52.8)
- C1, C2, C3, C6: value 100uF -> 100nF
- R4: value 100K -> 10K
- SW1: value SW_SPST_G -> SW_SPDT; footprint Nour_KB:EVQP9102W -> Nour_KB:CSS-1211TB
- moved Y2 191.9 mm to (6.75, 40.5), turned to -90 degrees
- moved C12 187.8 mm to (3.25, 38.8), turned to -90 degrees
- moved C13 180.4 mm to (10.2, 42.2), turned to -90 degrees
- moved R7 178.3 mm to (10.2, 38.8), turned to -90 degrees
- moved C11 166.2 mm to (13.0, 42.2), turned to -90 degrees
- moved C10 163.2 mm to (15.0, 42.2), turned to -90 degrees
- moved Y1 159.3 mm to (13.8, 38.8), turned to 180 degrees
- moved C7 125.6 mm to (18.8, 3.68)
- moved U2 125.0 mm to (18.8, 6.68)
- moved R4 124.8 mm to (6.30, 21.9), turned to 180 degrees
- moved C8 123.3 mm to (18.8, 9.68)
- moved SW1 122.4 mm to (2.75, 18.5), turned to -90 degrees
- moved R1 94.1 mm to (6.80, 32.5), turned to 90 degrees
- moved R5 91.4 mm to (6.90, 29.7), turned to 180 degrees
- moved R10 89.9 mm to (25.8, 8.50)
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Connections:
- IC1 pad 10: /core/LED.SW_RED2 -> /core/LED.SW_RED1
- IC1 pad 11: /core/LED.SW_BLUE2 -> /core/LED.SW_BLUE1
- IC1 pad 13: /core/LED.SW_GREEN1 -> /core/LED.SW_GREEN2
- IC1 pad 14: /core/LED.SW_RED1 -> /core/LED.SW_RED2
- IC1 pad 15: /core/LED.SW_BLUE1 -> /core/LED.SW_BLUE2
- IC1 pad 2: /core/LED.SW_GREEN4 -> /core/LED.SW_GREEN3
- IC1 pad 3: /core/LED.SW_RED4 -> /core/LED.SW_RED3
- IC1 pad 4: /core/LED.SW_BLUE4 -> /core/LED.SW_BLUE3
- IC1 pad 6: /core/LED.SW_GREEN3 -> /core/LED.SW_GREEN4
- IC1 pad 7: /core/LED.SW_RED3 -> /core/LED.SW_RED4
- IC1 pad 8: /core/LED.SW_BLUE3 -> /core/LED.SW_BLUE4
- IC1 pad 9: /core/LED.SW_GREEN2 -> /core/LED.SW_GREEN1
- J4 pad A5: Net-(J3-PadA5) -> Net-(J4-PadA5)
- J4 pad B5: Net-(J3-PadB5) -> Net-(J4-PadB5)
- J5 pad 3: /core/USART.RX -> /core/USART.TX
- J5 pad 4: /core/USART.TX -> /core/USART.RX
- R4 pad 1: GND -> /core/BOOT0
- R4 pad 2: /core/BOOT0 -> Net-(R4-Pad2)
- SW1 pad 1: /core/BOOT0 -> GND
- SW1 pad 2: VCC -> Net-(R4-Pad2)
- SW1 pad 3: /core/BOOT0 -> VCC
- U1 pad A2: /core/KEY.ROW10 -> /core/KEY.ROW6
- U1 pad A3: /core/KEY.ROW6 -> /core/KEY.ROW7
- U1 pad A4: /core/KEY.ROW7 -> /core/KEY.ROW2
- U1 pad A6: /core/KEY.COL2 -> /core/KEY.ROW3
- U1 pad B5: /core/KEY.COL1 -> /core/KEY.ROW4
- U1 pad B7: /core/KEY.ROW2 -> /core/KEY.COL5
- U1 pad C1: /core/KEY.COL10 -> /core/KEY.ROW8
- U1 pad C4: /core/KEY.ROW8 -> /core/KEY.ROW1
- U1 pad D1: /core/KEY.ROW9 -> /core/KEY.COL6
- U1 pad D3: /core/KEY.ROW4 -> /core/KEY.ROW9
- U1 pad E2: /core/KEY.COL9 -> /core/KEY.ROW10
- U1 pad E3: /core/KEY.ROW5 -> /core/KEY.COL7
- U1 pad E7: /core/KEY.ROW1 -> /core/KEY.ROW5
- U1 pad F1: /core/KEY.COL7 -> /core/KEY.COL10
- U1 pad F2: /core/KEY.COL6 -> /core/KEY.COL2
- U1 pad G1: /core/KEY.COL5 -> /core/KEY.COL9
- U1 pad G3: /core/KEY.COL3 -> /core/KEY.COL1
- U1 pad G4: /core/KEY.ROW3 -> /core/KEY.COL3
Routing:
- net /core/USART.RX: track 0.00 -> 117.2 mm, vias 0 -> 2
- net /core/D+: track 0.00 -> 102.7 mm, vias 0 -> 2
- net /core/D-: track 0.00 -> 101.7 mm, vias 0 -> 1
- net VBUS: track 0.00 -> 96.2 mm, vias 0 -> 1
- net /core/USART.TX: track 0.00 -> 80.8 mm, vias 0 -> 2
- net GND: track 0.00 -> 64.8 mm, vias 0 -> 31
- net /core/KEY.COL1: track 0.00 -> 47.3 mm, vias 0 -> 1
- net /core/KEY.COL2: track 0.00 -> 47.1 mm, vias 0 -> 2
- net VCC: track 0.00 -> 46.8 mm, vias 0 -> 2
- net /core/~{RST}: track 0.00 -> 45.3 mm, vias 0 -> 3
- net /core/KEY.COL10: track 0.00 -> 43.9 mm, vias 0 -> 1
- net /core/KEY.COL3: track 0.00 -> 43.5 mm, vias 0 -> 1
- net /core/KEY.COL4: track 0.00 -> 42.5 mm, vias 0 -> 2
- net /core/KEY.COL9: track 0.00 -> 42.2 mm, vias 0 -> 1
- net /core/KEY.COL8: track 0.00 -> 40.6 mm, vias 0 -> 1
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- added copper zone on B.Cu, net GND
- added copper zone on F.Cu, net VCC
Other:
- board size 304 x 240 mm -> 414.5 x 281.2 mm
