File: pcb/NourK/core.kicad_sch (KiCad schematic)
At the start: 49 parts, among them IC1 IS31FL3733B-QFLS4-TR, J1 SJ-435107RS, J2 Conn_ARM_JTAG_SWD_10, J3 USB_C_Receptacle_USB2.0, J4 USB_C_Receptacle_USB2.0, J5 SJ-435107RS, SW1 SW_SPDT, SW2 SW_SPST_G, U1 STM32L082CZYx, U2 AP2112K-3.3, U4 NourK_Core, Y1 32.768KHz, Y2 8MHz

Commit message: Complete wiring
Connections:
- net LED.SW_BLUE1: now also IC1.15 (SW12), U4.8 (LED_SW_BLUE2); no longer IC1.11 (SW9), U4.43 (LED_SW_BLUE1)
- net LED.SW_BLUE2: now also IC1.11 (SW9), U4.43 (LED_SW_BLUE1); no longer IC1.15 (SW12), U4.8 (LED_SW_BLUE2)
- net LED.SW_BLUE3: now also IC1.8 (SW6); no longer IC1.4 (SW3)
- net LED.SW_BLUE4: now also IC1.4 (SW3), U4.31 (LED_SW_GREEN4); no longer IC1.8 (SW6), U4.30 (LED_SW_BLUE4)
- net LED.SW_GREEN1: now also IC1.13 (SW10), U4.7 (LED_SW_GREEN2); no longer IC1.9 (SW7), U4.42 (LED_SW_GREEN1)
- net LED.SW_GREEN2: now also IC1.9 (SW7), U4.42 (LED_SW_GREEN1); no longer IC1.13 (SW10), U4.7 (LED_SW_GREEN2)
- net LED.SW_GREEN3: now also IC1.6 (SW4); no longer IC1.2 (SW1)
- net LED.SW_GREEN4: now also IC1.2 (SW1), U4.19 (LED_SW_RED4); no longer IC1.6 (SW4), U4.31 (LED_SW_GREEN4)
- net LED.SW_RED1: now also IC1.14 (SW11), U4.41 (LED_SW_RED2); no longer IC1.10 (SW8), U4.6 (LED_SW_RED1)
- net LED.SW_RED2: now also IC1.10 (SW8), U4.6 (LED_SW_RED1); no longer IC1.14 (SW11), U4.41 (LED_SW_RED2)
- net LED.SW_RED3: now also IC1.7 (SW5); no longer IC1.3 (SW2)
- net LED.SW_RED4: now also IC1.3 (SW2), U4.30 (LED_SW_BLUE4); no longer IC1.7 (SW5), U4.19 (LED_SW_RED4)
- net VCC: now also J1.6, J5.6; no longer J1.2, J5.2
- net at J1.5: now also J1.2
- net at J5.5: now also J5.2
- no-connect marks 14 -> 10
