File: pcb/valkyrie/core.kicad_sch (KiCad schematic)
At the start: 49 parts, among them IC1 IS31FL3733B-QFLS4-TR, J1 SJ-435107RS, J2 Conn_ARM_JTAG_SWD_10, J3 USB_C_Receptacle_USB2.0, J4 USB_C_Receptacle_USB2.0, J5 SJ-435107RS, SW1 SW_SPDT, SW2 SW_SPST_G, U1 STM32L082CZYx, U2 AP2112K-3.3, U4 NourK_Core, Y1 32.768KHz, Y2 8MHz

Commit message: Rename project
Parts:
- U4: footprint Nour_KB:NourKB_Core_2 -> Nour_KB:Nour_Core; symbol Nour_KB:NourK_Core_3 -> Nour_KB:Nour_Core
Changed lines of the file:
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@@
     (pin "2")
   )
-  (symbol (lib_id "Nour_KB:NourK_Core_3") (at 349.25 66.04 90) (unit 1)
+  (symbol (lib_id "Nour_KB:Nour_Core") (at 349.25 66.04 90) (unit 1)
     (in_bom no) (on_board yes) (fields_autoplaced)
     (property "Reference" "U4" (id 0) (at 349.25 25.561 90))
     (property "Value" "NourK_Core" (id 1) (at 349.25 28.0979 90))
-    (property "Footprint" "Nour_KB:NourKB_Core_2" (id 2) (at 367.03 38.1 0)
+    (property "Footprint" "Nour_KB:Nour_Core" (id 2) (at 367.03 38.1 0)
       (effects (font (size 1.27 1.27)) hide)
     )
