File: pcb/valkyrie/rhs.kicad_sch (KiCad schematic)
At the start: 1 part, among them U3 NourK_Core

Commit message: Rename project
Parts:
- U3: footprint Nour_KB:NourKB_Core_2 -> Nour_KB:Nour_Core; symbol Nour_KB:NourK_Core_3 -> Nour_KB:Nour_Core
Changed lines of the file:
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@@
     (effects (font (size 1.27 1.27)) (justify left bottom))
   )
-  (symbol (lib_id "Nour_KB:NourK_Core_3") (at 158.75 101.6 0) (unit 1)
+  (symbol (lib_id "Nour_KB:Nour_Core") (at 158.75 101.6 0) (unit 1)
     (in_bom no) (on_board yes)
     (property "Reference" "U3" (id 0) (at 160.02 105.41 0)
@@
       (effects (font (size 1.27 1.27)) (justify right))
     )
-    (property "Footprint" "Nour_KB:NourKB_Core_2" (id 2) (at 186.69 119.38 0)
+    (property "Footprint" "Nour_KB:Nour_Core" (id 2) (at 186.69 119.38 0)
       (effects (font (size 1.27 1.27)) hide)
     )
